File: KTH_HIL-adapter_board_1.0/KTH_HIL-adapter_board_1.0.sch (KiCad schematic (older format))
At the start: 0 parts

Commit message: push new resistor (#2)
Parts:
- added R?: R, symbol Device:R
Changed lines of the file:
@@
 EESchema Schematic File Version 4
+LIBS:KTH_HIL-adapter_board_1.0-cache
 EELAYER 30 0
 EELAYER END
@@
 Comment4 ""
 $EndDescr
+$Comp
+L Device:R R?
+U 1 1 6323225A
+P 5475 3000
+F 0 "R?" H 5545 3046 50  0000 L CNN
+F 1 "R" H 5545 2955 50  0000 L CNN
+F 2 "" V 5405 3000 50  0001 C CNN
+F 3 "~" H 5475 3000 50  0001 C CNN
+	1    5475 3000
+	1    0    0    -1
+$EndComp
 $EndSCHEMATC
