File: ADAPTER_BOARD/KTH_HIL-adapter_board_1.0/HIL_ADAPTER_BOARD.sch (KiCad schematic (older format))
At the start: 4 parts, among them CN10 Conn_02x20_Odd_Even, CN11 Conn_02x36_Odd_Even, CN12 Conn_02x36_Odd_Even, CN7 Conn_02x20_Odd_Even

Commit message: fixed timer issue in routing
Connections:
- net HiL_595_Enable: now also CN12.52 (Pin_52); no longer CN11.37 (Pin_37)
- no-connect marks 135 -> 137
Changed lines of the file:
@@
 Text Notes 1400 2775 0    50   ~ 0
 (SPI1)
-Text Label 950  2375 0    50   ~ 0
-HiL_595_Enable
-Wire Wire Line
-	950  2375 1825 2375
 Text Label 3200 1875 2    50   ~ 0
 HiL_USR_LED1
@@
 NoConn ~ 2325 6500
 NoConn ~ 2325 6600
-NoConn ~ 2325 6700
 NoConn ~ 1825 6400
 NoConn ~ 1825 6500
@@
 Text Notes 3225 1900 0    50   ~ 0
 <-
-Text Notes 800  2400 0    50   ~ 0
-->
 Text Notes 800  2300 0    50   ~ 0
 ->
@@
 Text Notes 3225 2400 0    50   ~ 0
 <-
+Text Label 3200 6700 2    50   ~ 0
+HiL_595_Enable
+Wire Wire Line
+	3200 6700 2325 6700
+Text Notes 3225 6725 0    50   ~ 0
+<-
+NoConn ~ 1825 1975
+NoConn ~ 1825 2075
+NoConn ~ 1825 2375
 $EndSCHEMATC
